Commit message: chore: no joint tracjer

File: robots/a1_description/urdf/a1.urdf (robot description, URDF)
Before this commit: robot a1, 23 links, 22 joints
Joints:
- joint FL_calf_joint: limit lower=-2.69653369433 upper=-0.916297857297 effort=33.5 velocity=21 -> lower=-2.69653369433 upper=0 effort=33.5 velocity=21
- joint FR_calf_joint: limit lower=-2.69653369433 upper=-0.916297857297 effort=33.5 velocity=21 -> lower=-2.69653369433 upper=0 effort=33.5 velocity=21
- joint RL_calf_joint: limit lower=-2.69653369433 upper=-0.916297857297 effort=33.5 velocity=21 -> lower=-2.69653369433 upper=0 effort=33.5 velocity=21
- joint RR_calf_joint: limit lower=-2.69653369433 upper=-0.916297857297 effort=33.5 velocity=21 -> lower=-2.69653369433 upper=0 effort=33.5 velocity=21

Commit message: chore: lidar sim

File: robots/a1_description/urdf/a1.urdf (robot description, URDF)
Before this commit: robot a1, 23 links, 22 joints
Links:
- added link rplidar; visual mesh filename=package://a1_description/meshes/rplidar.dae
Joints:
- added joint rplidar_fixed: type fixed, parent trunk, child rplidar, origin xyz=0 0 0.14 rpy=0 0 0

File: robots/a1_description/xacro/gazebo.xacro (robot description, xacro)
@@ -58,36 +58,36 @@
     <gazebo reference="FR_calf">
         <sensor name="FR_foot_contact" type="contact">
-        <update_rate>100</update_rate>
-        <plugin name="contactPlugin" filename="libunitreeFootContactPlugin.so"/>
-        <contact>
-            <collision>FR_calf_fixed_joint_lump__FR_foot_collision_1</collision>
-        </contact>
+            <update_rate>100</update_rate>
+            <plugin name="contactPlugin" filename="libunitreeFootContactPlugin.so"/>
+            <contact>
+                <collision>FR_calf_fixed_joint_lump__FR_foot_collision_1</collision>
+            </contact>
         </sensor>
     </gazebo>
     <gazebo reference="FL_calf">
         <sensor name="FL_foot_contact" type="contact">
-        <update_rate>100</update_rate>
-        <plugin name="contactPlugin" filename="libunitreeFootContactPlugin.so"/>
-        <contact>
-            <collision>FL_calf_fixed_joint_lump__FL_foot_collision_1</collision>
-        </contact>
+            <update_rate>100</update_rate>
+            <plugin name="contactPlugin" filename="libunitreeFootContactPlugin.so"/>
+            <contact>
+                <collision>FL_calf_fixed_joint_lump__FL_foot_collision_1</collision>
+            </contact>
         </sensor>
     </gazebo>
     <gazebo reference="RR_calf">
         <sensor name="RR_foot_contact" type="contact">
-        <update_rate>100</update_rate>
-        <plugin name="contactPlugin" filename="libunitreeFootContactPlugin.so"/>
-        <contact>
-            <collision>RR_calf_fixed_joint_lump__RR_foot_collision_1</collision>
-        </contact>
+            <update_rate>100</update_rate>
+            <plugin name="contactPlugin" filename="libunitreeFootContactPlugin.so"/>
+            <contact>
+                <collision>RR_calf_fixed_joint_lump__RR_foot_collision_1</collision>
+            </contact>
         </sensor>
     </gazebo>
     <gazebo reference="RL_calf">
         <sensor name="RL_foot_contact" type="contact">
-        <update_rate>100</update_rate>
-        <plugin name="contactPlugin" filename="libunitreeFootContactPlugin.so"/>
-        <contact>
-            <collision>RL_calf_fixed_joint_lump__RL_foot_collision_1</collision>
-        </contact>
+            <update_rate>100</update_rate>
+            <plugin name="contactPlugin" filename="libunitreeFootContactPlugin.so"/>
+            <contact>
+                <collision>RL_calf_fixed_joint_lump__RL_foot_collision_1</collision>
+            </contact>
         </sensor>
     </gazebo>
@@ -128,6 +128,6 @@
         <mu1>0.2</mu1>
         <mu2>0.2</mu2>
-        <kp  value="1000000.0"/>
-        <kd  value="1.0"/>
+        <kp value="1000000.0"/>
+        <kd value="1.0"/>
     </gazebo>
     <gazebo reference="stick_link">
@@ -152,6 +152,6 @@
         <self_collide>1</self_collide>
         <material>Gazebo/DarkGrey</material>
-        <kp  value="1000000.0"/>
-        <kd  value="1.0"/>
+        <kp value="1000000.0"/>
+        <kd value="1.0"/>
     </gazebo>
     <gazebo reference="FL_calf">
@@ -165,6 +165,6 @@
         <self_collide>1</self_collide>
         <material>Gazebo/DarkGrey</material>
-        <kp  value="1000000.0"/>
-        <kd  value="1.0"/>
+        <kp value="1000000.0"/>
+        <kd value="1.0"/>
     </gazebo>
     <!-- FR leg -->
@@ -179,6 +179,6 @@
         <self_collide>1</self_collide>
         <material>Gazebo/DarkGrey</material>
-        <kp  value="1000000.0"/>
-        <kd  value="1.0"/>
+        <kp value="1000000.0"/>
+        <kd value="1.0"/>
     </gazebo>
     <gazebo reference="FR_calf">
@@ -192,6 +192,6 @@
         <self_collide>1</self_collide>
         <material>Gazebo/DarkGrey</material>
-        <kp  value="1000000.0"/>
-        <kd  value="1.0"/>
+        <kp value="1000000.0"/>
+        <kd value="1.0"/>
     </gazebo>
     <!-- RL leg -->
@@ -206,6 +206,6 @@
         <self_collide>1</self_collide>
         <material>Gazebo/DarkGrey</material>
-        <kp  value="1000000.0"/>
-        <kd  value="1.0"/>
+        <kp value="1000000.0"/>
+        <kd value="1.0"/>
     </gazebo>
     <gazebo reference="RL_calf">
@@ -219,6 +219,6 @@
         <self_collide>1</self_collide>
         <material>Gazebo/DarkGrey</material>
-        <kp  value="1000000.0"/>
-        <kd  value="1.0"/>
+        <kp value="1000000.0"/>
+        <kd value="1.0"/>
     </gazebo>
     <!-- RR leg -->
@@ -233,6 +233,6 @@
         <self_collide>1</self_collide>
         <material>Gazebo/DarkGrey</material>
-        <kp  value="1000000.0"/>
-        <kd  value="1.0"/>
+        <kp value="1000000.0"/>
+        <kd value="1.0"/>
     </gazebo>
     <gazebo reference="RR_calf">
@@ -246,6 +246,50 @@
         <self_collide>1</self_collide>
         <material>Gazebo/DarkGrey</material>
-        <kp  value="1000000.0"/>
-        <kd  value="1.0"/>
-    </gazebo>
+        <kp value="1000000.0"/>
+        <kd value="1.0"/>
+    </gazebo>
+    <!-- <gazebo reference="">
+        <material>Gazebo/Indigo</material>
+        <sensor type="depth" name="realsense_R200">
+            <always_on>true</always_on>
+            <visualize>false</visualize>
+            <camera>
+                <horizontal_fov>1.5184</horizontal_fov>
+                <image>
+                    <width>470</width>
+                    <height>270</height>
+                    <format>R8G8B8</format>
+                </image>
+                <depth_camera></depth_camera>
+                <clip>
+                    <near>0.03</near>
+                    <far>4</far>
+                </clip>
+            </camera>
+            <plugin name="camera_controller" filename="libgazebo_ros_openni_kinect.so">
+                <baseline>0.2</baseline>
+                <alwaysOn>true</alwaysOn>
+                <updateRate>15.0</updateRate>
+                <cameraName>d435</cameraName>
+                <frameName>depth_camera_link</frameName>
+                <imageTopicName>rgb/image_raw</imageTopicName>
+                <depthImageTopicName>depth/image_raw</depthImageTopicName>
+                <pointCloudTopicName>depth/points</pointCloudTopicName>
+                <cameraInfoTopicName>rgb/camera_info</cameraInfoTopicName>
+                <depthImageCameraInfoTopicName>depth/camera_info</depthImageCameraInfoTopicName>
+                <pointCloudCutoff>0.4</pointCloudCutoff>
+                <hackBaseline>0.07</hackBaseline>
+                <distortionK1>0.0</distortionK1>
+                <distortionK2>0.0</distortionK2>
+                <distortionK3>0.0</distortionK3>
+                <distortionT1>0.0</distortionT1>
+                <distortionT2>0.0</distortionT2>
+                <CxPrime>0.0</CxPrime>
+                <Cx>0.0</Cx>
+                <Cy>0.0</Cy>
+                <focalLength>0</focalLength>
+                <hackBaseline>0</hackBaseline>
+            </plugin>
+        </sensor>
+    </gazebo> -->
 </robot>

Commit message: chore: relocate rgbd camera

File: robots/a1_description/urdf/a1.urdf (robot description, URDF)
Before this commit: robot a1, 24 links, 23 joints
Links:
- added link d435
- added link d435_optical
Joints:
- added joint d435_fixed: type fixed, parent trunk, child d435, origin xyz=0.25 0 0 rpy=0 0 0
- added joint d435_optical_fixed: type fixed, parent d435, child d435_optical, origin xyz=0 0 0 rpy=-1.57079632679 0 -1.57079632679
- joint imu_joint: origin xyz=0 0 0 rpy=0 0 0 -> xyz=0 0 -0.1936 rpy=0 0 0
- joint rplidar_fixed: origin xyz=0 0 0.14 rpy=0 0 0 -> xyz=0 0 0.175 rpy=0 0 0

File: robots/a1_description/xacro/gazebo.xacro (robot description, xacro)
@@ -249,47 +249,3 @@
         <kd value="1.0"/>
     </gazebo>
-    <!-- <gazebo reference="">
-        <material>Gazebo/Indigo</material>
-        <sensor type="depth" name="realsense_R200">
-            <always_on>true</always_on>
-            <visualize>false</visualize>
-            <camera>
-                <horizontal_fov>1.5184</horizontal_fov>
-                <image>
-                    <width>470</width>
-                    <height>270</height>
-                    <format>R8G8B8</format>
-                </image>
-                <depth_camera></depth_camera>
-                <clip>
-                    <near>0.03</near>
-                    <far>4</far>
-                </clip>
-            </camera>
-            <plugin name="camera_controller" filename="libgazebo_ros_openni_kinect.so">
-                <baseline>0.2</baseline>
-                <alwaysOn>true</alwaysOn>
-                <updateRate>15.0</updateRate>
-                <cameraName>d435</cameraName>
-                <frameName>depth_camera_link</frameName>
-                <imageTopicName>rgb/image_raw</imageTopicName>
-                <depthImageTopicName>depth/image_raw</depthImageTopicName>
-                <pointCloudTopicName>depth/points</pointCloudTopicName>
-                <cameraInfoTopicName>rgb/camera_info</cameraInfoTopicName>
-                <depthImageCameraInfoTopicName>depth/camera_info</depthImageCameraInfoTopicName>
-                <pointCloudCutoff>0.4</pointCloudCutoff>
-                <hackBaseline>0.07</hackBaseline>
-                <distortionK1>0.0</distortionK1>
-                <distortionK2>0.0</distortionK2>
-                <distortionK3>0.0</distortionK3>
-                <distortionT1>0.0</distortionT1>
-                <distortionT2>0.0</distortionT2>
-                <CxPrime>0.0</CxPrime>
-                <Cx>0.0</Cx>
-                <Cy>0.0</Cy>
-                <focalLength>0</focalLength>
-                <hackBaseline>0</hackBaseline>
-            </plugin>
-        </sensor>
-    </gazebo> -->
 </robot>

Commit message: fix: better lidar pose

File: robots/a1_description/urdf/a1.urdf (robot description, URDF)
Before this commit: robot a1, 26 links, 25 joints
Joints:
- joint rplidar_fixed: origin xyz=0 0 0.175 rpy=0 0 0 -> xyz=0 0 0.14 rpy=0 0 0

Commit message: chore: no displaced imu

File: robots/a1_description/urdf/a1.urdf (robot description, URDF)
Before this commit: robot a1, 26 links, 25 joints
Joints:
- joint imu_joint: origin xyz=0 0 -0.1936 rpy=0 0 0 -> xyz=0 0 0 rpy=0 0 0
